Commit message: ✨ feat: 增加pytracik逆解模块

File: piper/piper.urdf (robot description, URDF)
Before this commit: robot piper, 10 links, 9 joints
Links:
- added link base_footprint; visual box size=0.01 0.01 0.01
Joints:
- added joint base_footprint_joint: type fixed, parent base_footprint, child base_link, origin xyz=0 0 0 rpy=0 0 0
